File: dac_mcp2716.kicad_sch (KiCad schematic)
At the start: 1 part, among them U6 MCP4716A0T-E_MAY

Commit message: pre pre production
Parts:
- U6: now left out of the parts list
Changed lines of the file:
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@@
   (paper "A4")
   (symbol (lib_id "2023-11-28_17-34-14:MCP4716A0T-E_MAY") (at 121.92 76.2 0) (unit 1)
-    (in_bom yes) (on_board yes) (dnp no) (fields_autoplaced)
+    (in_bom no) (on_board no) (dnp no) (fields_autoplaced)
     (property "Reference" "U6" (at 142.24 64.77 0)
       (effects (font (size 1.524 1.524)))
