File: mcu_buttons_leds.kicad_sch (KiCad schematic)
At the start: 48 parts, among them Q2 L8050QLT1G, Q3 L8050QLT1G, U1 W25Q128JVS, U7 ESP32-S2, Y1 Crystal_GND24

Commit message: added cp2102 schematics
Connections:
- net GPIO5: now reaches U7.10 (GPIO5/ADC1_CH4)
- net GPIO6: now reaches U7.11 (GPIO6/ADC1_CH5)
- net GPIO7: now reaches U7.12 (GPIO7/ADC1_CH6)
- net GPIO8: now reaches U7.13 (GPIO8/ADC1_CH7)
- net GPIO9: now reaches U7.14 (GPIO9/ADC1_CH8)
- net GPIO10: now reaches U7.15 (GPIO10/ADC1_CH9)
- net GPIO11: now reaches U7.16 (GPIO11/ADC2_CH0)
- net GPIO12: now reaches U7.17 (GPIO12/ADC2_CH1)
- net GPIO13: now reaches U7.18 (GPIO13/ADC2_CH2)
- net GPIO14: now reaches U7.19 (GPIO14/ADC2_CH3)
- net GPIO21: now reaches U7.28 (GPIO21)
- net GPIO33: now reaches U7.37 (GPIO33)
- net GPIO34: now reaches U7.38 (GPIO34)
- net GPIO35: now reaches U7.39 (GPIO35)
- net GPIO36: now reaches U7.40 (GPIO36)
- net GPIO37: now reaches U7.41 (GPIO37)
- net GPIO38: now reaches U7.42 (GPIO38)
- net GPIO1: now reaches U7.6 (GPIO1/ADC1_CH0)
- net GPIO2: now reaches U7.7 (GPIO2/ADC1_CH1)
- net GPIO3: now reaches U7.8 (GPIO3/ADC1_CH2)
- net GPIO4: now reaches U7.9 (GPIO4/ADC1_CH3)
- net ESP_RX renamed CP2102_TX
- net ESP_TX renamed CP2102_RX
- net USB_OTG_DN renamed USB_OTG_N
- net USB_OTG_DP renamed USB_OTG_P
- no-connect marks 4 -> 9
Other:
- note added: "CHECK THIS AGAIN!"
Changed lines of the file:
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@@
   )
   (no_connect (at 86.36 137.16))
+  (no_connect (at 80.01 124.46))
   (no_connect (at 86.36 109.22))
   (no_connect (at 162.56 175.26))
+  (no_connect (at 80.01 132.08))
+  (no_connect (at 80.01 129.54))
+  (no_connect (at 86.36 160.02))
   (no_connect (at 86.36 111.76))
+  (no_connect (at 80.01 127))
   (wire (pts (xy 212.09 139.7) (xy 217.17 139.7))
     (stroke (width 0) (type default))
@@
     (stroke (width 0) (type default))
   )
+  (wire (pts (xy 80.01 124.46) (xy 86.36 124.46))
+    (stroke (width 0) (type default))
+  )
   (wire (pts (xy 162.56 157.48) (xy 180.34 157.48))
     (stroke (width 0) (type default))
@@
     (stroke (width 0) (type default))
   )
+  (wire (pts (xy 162.56 101.6) (xy 180.34 101.6))
+    (stroke (width 0) (type default))
+  )
   (wire (pts (xy 25.4 97.79) (xy 25.4 100.33))
     (stroke (width 0) (type default))
@@
     (stroke (width 0) (type default))
   )
+  (wire (pts (xy 80.01 127) (xy 86.36 127))
+    (stroke (width 0) (type default))
+  )
   (wire (pts (xy 220.98 132.08) (xy 240.03 132.08))
     (stroke (width 0) (type default))
   )
+  (wire (pts (xy 80.01 132.08) (xy 86.36 132.08))
+    (stroke (width 0) (type default))
+  )
   (wire (pts (xy 162.56 137.16) (xy 180.34 137.16))
     (stroke (width 0) (type default))
@@
     (stroke (width 0) (type default))
   )
-  (wire (pts (xy 162.56 101.6) (xy 180.34 101.6))
-    (stroke (width 0) (type default))
-  )
   (wire (pts (xy 255.27 144.78) (xy 257.81 144.78))
     (stroke (width 0) (type default))
@@
   )
   (wire (pts (xy 106.68 50.8) (xy 106.68 55.88))
+    (stroke (width 0) (type default))
+  )
+  (wire (pts (xy 80.01 129.54) (xy 86.36 129.54))
     (stroke (width 0) (type default))
   )
@@
     (effects (font (size 1.27 1.27)) (justify left bottom))
   )
+  (text "CHECK THIS AGAIN!" (at 38.1 156.21 0)
+    (effects (font (size 1.27 1.27)) (justify left bottom))
+  )
   (text "XOUT" (at 45.72 114.3 0)
     (effects (font (size 1.27 1.27)) (justify left bottom))
   )
   (text "do not use gpio45 \nit is strapping pin for\nselect flash voltage"
-    (at 147.32 186.69 0)
+    (at 153.67 185.42 0)
     (effects (font (size 1.27 1.27)) (justify left bottom))
   )
@@
     (effects (font (size 1.27 1.27) (thickness 0.254) bold) (justify left bottom))
   )
-  (text "Boot strapping pin N3" (at 147.32 180.34 0)
+  (text "Boot strapping pin N3" (at 165.1 176.53 0)
     (effects (font (size 1.27 1.27)) (justify left bottom))
   )
@@
     (effects (font (size 1.27 1.27)) (justify left bottom))
   )
-  (text "ESP protection diode on global power input?\n" (at 223.52 40.64 0)
+  (text "ESP protection diode on global power input?\n" (at 140.97 33.02 0)
     (effects (font (size 1.27 1.27)) (justify left bottom))
   )
@@
     (effects (font (size 1.27 1.27)) (justify left bottom))
   )
+  (label "GPIO14" (at 180.34 149.86 0) (fields_autoplaced)
+    (effects (font (size 1.27 1.27)) (justify left bottom))
+  )
+  (label "GPIO13" (at 180.34 147.32 0) (fields_autoplaced)
+    (effects (font (size 1.27 1.27)) (justify left bottom))
+  )
   (label "CHIP_EN" (at 275.59 81.28 90) (fields_autoplaced)
     (effects (font (size 1.27 1.27)) (justify left bottom))
   )
+  (label "GPIO4" (at 180.34 124.46 0) (fields_autoplaced)
+    (effects (font (size 1.27 1.27)) (justify left bottom))
+  )
   (label "CIO0_BTN" (at 245.11 83.82 90) (fields_autoplaced)
     (effects (font (size 1.27 1.27)) (justify left bottom))
   )
+  (label "GPIO7" (at 180.34 132.08 0) (fields_autoplaced)
+    (effects (font (size 1.27 1.27)) (justify left bottom))
+  )
+  (label "GPIO8" (at 180.34 134.62 0) (fields_autoplaced)
+    (effects (font (size 1.27 1.27)) (justify left bottom))
+  )
+  (label "GPIO3" (at 180.34 121.92 0) (fields_autoplaced)
+    (effects (font (size 1.27 1.27)) (justify left bottom))
+  )
+  (label "GPIO33" (at 180.34 160.02 0) (fields_autoplaced)
+    (effects (font (size 1.27 1.27)) (justify left bottom))
+  )
+  (label "GPIO6" (at 180.34 129.54 0) (fields_autoplaced)
+    (effects (font (size 1.27 1.27)) (justify left bottom))
+  )
+  (label "GPIO12" (at 180.34 144.78 0) (fields_autoplaced)
+    (effects (font (size 1.27 1.27)) (justify left bottom))
+  )
   (label "CIO0_BTN" (at 257.81 144.78 0) (fields_autoplaced)
     (effects (font (size 1.27 1.27)) (justify left bottom))
   )
+  (label "GPIO38" (at 180.34 172.72 0) (fields_autoplaced)
+    (effects (font (size 1.27 1.27)) (justify left bottom))
+  )
+  (label "GPIO10" (at 180.34 139.7 0) (fields_autoplaced)
+    (effects (font (size 1.27 1.27)) (justify left bottom))
+  )
   (label "CHIP_EN" (at 74.93 104.14 0) (fields_autoplaced)
+    (effects (font (size 1.27 1.27)) (justify left bottom))
+  )
+  (label "GPIO34" (at 180.34 162.56 0) (fields_autoplaced)
+    (effects (font (size 1.27 1.27)) (justify left bottom))
+  )
+  (label "GPIO37" (at 180.34 170.18 0) (fields_autoplaced)
     (effects (font (size 1.27 1.27)) (justify left bottom))
   )
@@
     (effects (font (size 1.27 1.27)) (justify right bottom))
   )
+  (label "GPIO1" (at 180.34 116.84 0) (fields_autoplaced)
+    (effects (font (size 1.27 1.27)) (justify left bottom))
+  )
+  (label "GPIO5" (at 180.34 127 0) (fields_autoplaced)
+    (effects (font (size 1.27 1.27)) (justify left bottom))
+  )
+  (label "GPIO2" (at 180.34 119.38 0) (fields_autoplaced)
+    (effects (font (size 1.27 1.27)) (justify left bottom))
+  )
   (label "CHIP_EN" (at 259.08 116.84 0) (fields_autoplaced)
     (effects (font (size 1.27 1.27)) (justify left bottom))
   )
+  (label "GPIO21" (at 180.34 157.48 0) (fields_autoplaced)
+    (effects (font (size 1.27 1.27)) (justify left bottom))
+  )
+  (label "GPIO36" (at 180.34 167.64 0) (fields_autoplaced)
+    (effects (font (size 1.27 1.27)) (justify left bottom))
+  )
   (label "CIO0_BTN" (at 180.34 114.3 0) (fields_autoplaced)
     (effects (font (size 1.27 1.27)) (justify left bottom))
   )
+  (label "GPIO9" (at 180.34 137.16 0) (fields_autoplaced)
+    (effects (font (size 1.27 1.27)) (justify left bottom))
+  )
+  (label "GPIO35" (at 180.34 165.1 0) (fields_autoplaced)
+    (effects (font (size 1.27 1.27)) (justify left bottom))
+  )
+  (label "GPIO11" (at 180.34 142.24 0) (fields_autoplaced)
+    (effects (font (size 1.27 1.27)) (justify left bottom))
+  )
   (hierarchical_label "GND" (shape input) (at 34.29 151.13 90) (fields_autoplaced)
     (effects (font (size 1.27 1.27)) (justify left))
@@
     (effects (font (size 1.27 1.27)) (justify right))
   )
+  (hierarchical_label "CP2102_TX" (shape input) (at 180.34 101.6 0) (fields_autoplaced)
+    (effects (font (size 1.27 1.27)) (justify left))
+  )
   (hierarchical_label "RTS" (shape input) (at 212.09 139.7 180) (fields_autoplaced)
     (effects (font (size 1.27 1.27)) (justify right))
@@
     (effects (font (size 1.27 1.27)) (justify right))
   )
-  (hierarchical_label "USB_OTG_DP" (shape input) (at 180.34 106.68 0) (fields_autoplaced)
+  (hierarchical_label "USB_OTG_P" (shape input) (at 180.34 106.68 0) (fields_autoplaced)
     (effects (font (size 1.27 1.27)) (justify left))
   )
@@
     (effects (font (size 1.27 1.27)) (justify right))
   )
-  (hierarchical_label "ESP_RX" (shape input) (at 180.34 101.6 0) (fields_autoplaced)
+  (hierarchical_label "CP2102_RX" (shape input) (at 180.34 99.06 0) (fields_autoplaced)
     (effects (font (size 1.27 1.27)) (justify left))
   )
@@
     (effects (font (size 1.27 1.27)) (justify left))
   )
-  (hierarchical_label "USB_OTG_DN" (shape input) (at 180.34 109.22 0) (fields_autoplaced)
+  (hierarchical_label "USB_OTG_N" (shape input) (at 180.34 109.22 0) (fields_autoplaced)
     (effects (font (size 1.27 1.27)) (justify left))
   )
@@
     (effects (font (size 1.27 1.27)) (justify left))
   )
-  (hierarchical_label "ESP_TX" (shape input) (at 180.34 99.06 0) (fields_autoplaced)
-    (effects (font (size 1.27 1.27)) (justify left))
-  )

Commit message: schematics almost finished
Parts:
- removed Q2, Q3: L8050QLT1G, Package_TO_SOT_SMD:SOT-23, symbol Transistor_BJT:BC848W
- added D13, D14, D15, D16: LED, LED_SMD:LED_0805_2012Metric, symbol Device:LED
- added Q5, Q8: MMBT3904, Package_TO_SOT_SMD:SOT-23, symbol Transistor_BJT:MMBT3904
- added R42, R43, R44, R45: 5K, Resistor_SMD:R_0805_2012Metric, symbol Device:R
- added R46: 10K, Resistor_SMD:R_0805_2012Metric, symbol Device:R
- added S4: TS-1187A-B-A-B, TS-1187A-B-A-B:SW_TS-1187A-B-A-B, symbol TS-1187A-B-A-B:TS-1187A-B-A-B
- renumbered R15 to R27, R15 to R28
Connections:
- net 3V3: now also S4.C, S4.D
- net DTR: now also Q8.2 (E)
- net GND: now also D13.1 (K), D14.1 (K), D15.1 (K), D16.1 (K), R46.1
- net GPIO14: now also R46.2, S4.A, S4.B
- net RTS: now also Q5.2 (E)
- net at R15.1: now also Q5.1 (B)
- net at R21.1: now also Q8.3 (C)
- net at R20.1: now also Q5.3 (C)
- net at R16.1: now also Q8.1 (B)
- net GPIO1 renamed V_BAT_MEASURE
- net GPIO2 renamed GPIO_BUTTON_CHECK
- net GPIO3 renamed GPIO_POWEROFF
- net GPIO33: no longer names the net of U7.37 (GPIO33)
- net GPIO33: now also R42.1
- net GPIO34: no longer names the net of U7.38 (GPIO34)
- net GPIO34: now also R43.1
- net GPIO35: no longer names the net of U7.39 (GPIO35)
- net GPIO35: now also R44.1
- net GPIO36: no longer names the net of U7.40 (GPIO36)
- net GPIO36: now also R45.1
- new net: D16.2 (A), R45.2
- new net: D14.2 (A), R43.2
- new net: D13.2 (A), R42.2
- new net: D15.2 (A), R44.2
Other:
- note added: "Additional button with unknown purposes"
- note added: "MB add some voltage upper limit schematic, to save EEG device ???"
- note added: "https://docs.espressif.com/projects/esp-hardware-design-guidelines/en/latest/esp32s2/schematic-checklist.html#off-package-flash-and-psram"
- note added: "leds for battery level indication"
- moved on the sheet: AE2, C10, C11, C12, C13, C14, C15, C16, C17, C18, C19, C2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

Commit message: pre pre production
Parts:
- added J4, J5, J6: Conn_01x07_Pin, Connector_PinHeader_2.54mm:PinHeader_1x07_P2.54mm_Vertical, symbol Connector:Conn_01x07_Pin
- added OUTPUT1: Screw_Terminal_01x02, screws:screw-2-pin, symbol Connector:Screw_Terminal_01x02
- added R47: 0R, Resistor_SMD:R_0805_2012Metric, symbol Device:R
- AE2: footprint ESP_Antenna:ESPRESSIF_ESP32_MIFA_2.4GHz_Right -> RF_Antenna:Texas_SWRA117D_2.4GHz_Left
- D13, D14, D15, D16, R29, R30, R42, R43, R44, R45: now left out of the parts list
- L2, L3: footprint (none) -> Inductor_SMD:L_0805_2012Metric
- R6, R7, R8, R9: footprint (none) -> Resistor_SMD:R_0805_2012Metric
Connections:
- net 3V3: now also J5.1 (Pin_1), J5.2 (Pin_2), J5.3 (Pin_3), J5.4 (Pin_4), J5.5 (Pin_5), J5.6 (Pin_6), J5.7 (Pin_7)
- net DAC_OUT: now also R47.1
- net GND: now also J6.1 (Pin_1), J6.2 (Pin_2), J6.3 (Pin_3), J6.4 (Pin_4), J6.5 (Pin_5), J6.6 (Pin_6), J6.7 (Pin_7), OUTPUT1.2 (Pin_2)
- net GPIO10: now also J4.4 (Pin_4)
- net GPIO11: now also J4.5 (Pin_5)
- net GPIO12: now also J4.6 (Pin_6)
- net GPIO13: now also J4.7 (Pin_7)
- net GPIO7: now also J4.1 (Pin_1)
- net GPIO8: now also J4.2 (Pin_2)
- net GPIO9: now also J4.3 (Pin_3)
- net GPIO5 renamed DOUT
- net GPIO6 renamed PD_SCK
- new net: OUTPUT1.1 (Pin_1), R47.2
Other:
- note added: "Inductor L2 must be very powerful, like more than 500mA"
- note added: "for now usb otg excluded from board"
- moved on the sheet: C7, C8

Commit message: finished
Parts:
- removed D13, D14, D15, D16: LED, LED_SMD:LED_0805_2012Metric, symbol Device:LED
- removed R44, R45: 5K, Resistor_SMD:R_0805_2012Metric, symbol Device:R
- removed R47: 0R, Resistor_SMD:R_0805_2012Metric, symbol Device:R
- removed S1, S2, S4: TS-1187A-B-A-B, TS-1187A-B-A-B:SW_TS-1187A-B-A-B, symbol TS-1187A-B-A-B:TS-1187A-B-A-B
- added J7: Conn_01x04_Pin, Connector_PinHeader_2.54mm:PinHeader_1x04_P2.54mm_Vertical, symbol Connector:Conn_01x04_Pin
- added SW1, SW2, SW3: SW_DPST, Button_Switch_SMD:SW_Push_1P1T_NO_6x6mm_H9.5mm, symbol Switch:SW_DPST
- C17: value 10pF -> 1.2pF
- C18: value 10pF -> 1.8pF
- L3: value 2nH -> 2.4nH
- R42: value 5K -> 30K; now in the parts list
- R43: value 5K -> 10K; now in the parts list
Connections:
- net 3V3: now also J7.2 (Pin_2), SW1.2, SW1.4
- net DAC_OUT: now also OUTPUT1.1 (Pin_1), R42.2, R43.2; no longer U7.23 (GPIO17/ADC2_CH6/DAC_1)
- net GND: now also R43.1, J7.1 (Pin_1), SW2.1, SW2.3, SW3.2, SW3.4
- net GPIO14: now also SW1.1, SW1.3
- net GPIO36: now reaches U7.40 (GPIO36)
- net GPIO36: now also J7.4 (Pin_4)
- net GPIO34: now reaches U7.38 (GPIO34)
- net GPIO34: no longer R43.1
- net at C20.2, R18.1: now also SW2.2, SW2.4
- net at R42.1: now also U7.23 (GPIO17/ADC2_CH6/DAC_1); no longer U7.37 (GPIO33)
- net GPIO35: now reaches U7.39 (GPIO35)
- net GPIO35: now also J7.3 (Pin_3)
- net at C22.2, R22.1: now also SW3.1, SW3.3
- new net GPIO33: U7.37 (GPIO33)
Other:
- note added: "GPIO for some modding or debug"
- note added: "I dont know how to calculate matching circuit for RF :("
- note added: "I2C for OLED"
- note added: "OLED SCK"
- note added: "OLED SDA"
- note added: "SCK"
- note added: "SDA"
- note added: "https://microchip.my.site.com/s/article/Calculating-crystal-load-capacitor C1 = C2 = 2 * (CL - Cstray) Cstray ~ 5pf, CL - from xtal datasheet"
- note added: "https://www.will-kelsey.com/smith_chart/"
- note added: "ДОБАВИТЬ на выход ЦАП2 резисторный делитель напряжения!"
- note added: "расчет и выбор антенн https://www.ti.com/lit/an/swra161b/swra161b.pdf"
- note removed: "CHECK THIS AGAIN!"
- note removed: "MB add some voltage upper limit schematic, to save EEG device ???"
- note removed: "leds for battery level indication"
- moved on the sheet: J4, OUTPUT1

Commit message: minor fix
Other:
- note added: "MB make that resistors like 1 MOhm, to reduce output current?"
Changed lines of the file:
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@@
+    (effects (font (size 1.27 1.27)) (justify left bottom))
+  )
+  (text "MB make that resistors like 1 MOhm, to reduce output current?"
+    (at 243.84 172.72 0)
     (effects (font (size 1.27 1.27)) (justify left bottom))
   )
