File: tp4056.kicad_sch (KiCad schematic)
At the start: 1 part, among them U3 TP4056

Commit message: schematics almost finished
Parts:
- added BAT: Conn_01x02_Pin, Connector_PinHeader_2.54mm:PinHeader_1x02_P2.54mm_Vertical, symbol Connector:Conn_01x02_Pin
- added C24: 10uF, Capacitor_SMD:C_0805_2012Metric, symbol Device:C
- added C25, C29: 2uF, Capacitor_SMD:C_0805_2012Metric, symbol Device:C
- added C30: 100n, Capacitor_SMD:C_0805_2012Metric, symbol Device:C
- added D11, D12: SS54, Diode_SMD:D_SMA, symbol Diode:B340
- added D7: RED LED, Diode_SMD:D_0805_2012Metric, symbol Device:LED
- added D8: GREEN LED, Diode_SMD:D_0805_2012Metric, symbol Device:LED
- added D9: SS54, Diode_SMD:D_SMA, symbol Device:D_Schottky
- added Q4, Q6: AO3401A, Package_TO_SOT_SMD:SOT-23, symbol Transistor_FET:AO3401A
- added Q7: AO3400A, Package_TO_SOT_SMD:SOT-23, symbol Transistor_FET:AO3400A
- added R14, R23: 1K, Resistor_SMD:R_0805_2012Metric, symbol Device:R
- added R26: 1K5, Resistor_SMD:R_0805_2012Metric, symbol Device:R
- added R35, R38, R41: 100K, Resistor_SMD:R_0805_2012Metric, symbol Device:R
- added R36: 10K, Resistor_SMD:R_0805_2012Metric, symbol Device:R
- added R37: 30K, Resistor_SMD:R_0805_2012Metric, symbol Device:R
- added R39: 1M, Resistor_SMD:R_0805_2012Metric, symbol Device:R
- added R40: 100R, Resistor_SMD:R_0805_2012Metric, symbol Device:R
- added S3: TS-1187A-B-A-B, TS-1187A-B-A-B:SW_TS-1187A-B-A-B, symbol TS-1187A-B-A-B:TS-1187A-B-A-B
- added U8: TLV75733PDBV, Package_TO_SOT_SMD:SOT-23-5, symbol Regulator_Linear:TLV75733PDBV
Connections:
- net GND: now reaches U3.1 (TEMP)
- net GND: now also U3.3 (GND), U3.9 (EP), BAT.1 (Pin_1), C24.2, C25.2, C29.2, Q7.2 (S), R26.2, R35.2, R37.2, R39.2, R40.2, R41.2, U8.2 (GND)
- net at U3.2 (PROG): now also R26.1
- net C5V_USB: now reaches U3.4 (VCC)
- net C5V_USB: now also U3.8 (CE), C24.1, D7.2 (A), D8.2 (A), D9.2 (A), Q4.1 (G), R35.1
- net V_BAT: now reaches U3.5 (BAT)
- net V_BAT: now also BAT.2 (Pin_2), Q4.3 (D), R36.1
- net at U3.6 (~{STDBY}): now also R14.2
- net at U3.7 (~{CHRG}): now also R23.2
- new net: C30.2, D11.2 (A), Q6.1 (G), Q7.3 (D), R38.2
- new net: D8.1 (K), R14.1
- new net: D11.1 (K), D12.1 (K), S3.A, S3.B
- new net: D7.1 (K), R23.1
- new net: R40.1, S3.C, S3.D
- new net 3V3: C29.1, U8.5 (OUT)
- new net GPIO_BUTTON_CHECK: D12.2 (A)
- new net GPIO_POWEROFF: Q7.1 (G), R39.1
- new net POWER_EN: Q6.3 (D), R41.1, U8.3 (EN)
- new net V_BAT_MEASURE: R36.2, R37.1
- new net V_MIXED: C25.1, C30.1, D9.1 (K), Q4.2 (S), Q6.2 (S), R38.1, U8.1 (IN)
Other:
- note added: "D"
- note added: "Do we need that resistor?"
- note added: "G"
- note added: "LI-Po charger"
- note added: "Main power supply from Li-Po/USB to 3v3"
- note added: "Power selector scheme"
- note added: "S"
- note added: "Voltage divider to measure v batt on esp adc, to show to user"
- note added: "https://www.best-microcontroller-projects.com/dw01a.html"
- note added: "https://www.best-microcontroller-projects.com/tp4056.html"
- note added: "https://www.ti.com/lit/ds/symlink/tlv757p.pdf"
- note added: "must be pulled up"
- note added: "power on system"
- moved on the sheet: U3

Commit message: pre pre production
Parts:
- D7, D8: footprint Diode_SMD:D_0805_2012Metric -> LED_SMD:LED_0805_2012Metric
- U3: footprint Package_SO:SOP-8_3.9x4.9mm_P1.27mm -> TP4056:SOP127P600X175-9N
- renumbered BAT to BAT1
Changed lines of the file:
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@@
       (effects (font (size 1.27 1.27)) (justify right))
     )
-    (property "Footprint" "Diode_SMD:D_0805_2012Metric" (at 102.87 156.21 0)
+    (property "Footprint" "LED_SMD:LED_0805_2012Metric" (at 102.87 156.21 0)
       (effects (font (size 1.27 1.27)) hide)
     )
@@
       (effects (font (size 1.27 1.27)) (justify right))
     )
-    (property "Footprint" "Diode_SMD:D_0805_2012Metric" (at 102.87 163.83 0)
+    (property "Footprint" "LED_SMD:LED_0805_2012Metric" (at 102.87 163.83 0)
       (effects (font (size 1.27 1.27)) hide)
     )
@@
       (effects (font (size 1.27 1.27)))
     )
-    (property "Footprint" "Package_SO:SOP-8_3.9x4.9mm_P1.27mm" (at 71.12 158.75 0)
+    (property "Footprint" "TP4056:SOP127P600X175-9N" (at 71.12 158.75 0)
       (effects (font (size 1.27 1.27)) (justify bottom) hide)
     )
@@
   (symbol (lib_id "Connector:Conn_01x02_Pin") (at 124.46 161.29 180) (unit 1)
     (in_bom yes) (on_board yes) (dnp no) (fields_autoplaced)
-    (property "Reference" "BAT" (at 125.73 158.75 0)
+    (property "Reference" "BAT1" (at 125.73 158.75 0)
       (effects (font (size 1.27 1.27)) (justify right))
     )
@@
       (project "grip_strength_meter"
         (path "/1f4b217c-5456-4c03-a123-3ef9839449c6/4e936500-8830-4ef1-9c08-090defb3e135"
-          (reference "BAT") (unit 1)
-        )
-      )
+          (reference "BAT1") (unit 1)
+        )
+      )

Commit message: finished
Parts:
- removed S3: TS-1187A-B-A-B, TS-1187A-B-A-B:SW_TS-1187A-B-A-B, symbol TS-1187A-B-A-B:TS-1187A-B-A-B
- added SW4: SW_DPST, Button_Switch_SMD:SW_Push_1P1T_NO_6x6mm_H9.5mm, symbol Switch:SW_DPST
- C30: value 100n -> 100nF
Connections:
- net at D11.1 (K), D12.1 (K): now also SW4.2, SW4.4
- net at R40.1: now also SW4.1, SW4.3
Other:
- moved on the sheet: R39, R40
Changed lines of the file:
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@@
   (junction (at 91.44 140.97) (diameter 0) (color 0 0 0 0)
   )
+  (junction (at 106.68 60.96) (diameter 0) (color 0 0 0 0)
+  )
   (junction (at 153.67 137.16) (diameter 0) (color 0 0 0 0)
   )
@@
   (junction (at 113.03 151.13) (diameter 0) (color 0 0 0 0)
   )
+  (junction (at 106.68 71.12) (diameter 0) (color 0 0 0 0)
+  )
   (junction (at 148.59 137.16) (diameter 0) (color 0 0 0 0)
   )
@@
     (stroke (width 0) (type default))
   )
-  (wire (pts (xy 74.93 54.61) (xy 96.52 54.61))
+  (wire (pts (xy 101.6 60.96) (xy 106.68 60.96))
+    (stroke (width 0) (type default))
+  )
+  (wire (pts (xy 74.93 54.61) (xy 99.06 54.61))
     (stroke (width 0) (type default))
   )
@@
     (stroke (width 0) (type default))
   )
+  (wire (pts (xy 106.68 71.12) (xy 111.76 71.12))
+    (stroke (width 0) (type default))
+  )
   (wire (pts (xy 93.98 107.95) (xy 93.98 109.22))
     (stroke (width 0) (type default))
@@
     (stroke (width 0) (type default))
   )
+  (wire (pts (xy 101.6 71.12) (xy 106.68 71.12))
+    (stroke (width 0) (type default))
+  )
   (wire (pts (xy 90.17 151.13) (xy 113.03 151.13))
     (stroke (width 0) (type default))
@@
     (stroke (width 0) (type default))
   )
+  (wire (pts (xy 101.6 73.66) (xy 101.6 71.12))
+    (stroke (width 0) (type default))
+  )
   (wire (pts (xy 52.07 41.91) (xy 57.15 41.91))
     (stroke (width 0) (type default))
@@
     (stroke (width 0) (type default))
   )
-  (wire (pts (xy 95.25 73.66) (xy 101.6 73.66))
+  (wire (pts (xy 91.44 73.66) (xy 101.6 73.66))
     (stroke (width 0) (type default))
   )
@@
     (stroke (width 0) (type default))
   )
+  (wire (pts (xy 101.6 58.42) (xy 101.6 60.96))
+    (stroke (width 0) (type default))
+  )
   (wire (pts (xy 59.69 73.66) (xy 67.31 73.66))
     (stroke (width 0) (type default))
@@
     (stroke (width 0) (type default))
   )
-  (wire (pts (xy 74.93 60.96) (xy 74.93 66.04))
-    (stroke (width 0) (type default))
-  )
-  (wire (pts (xy 95.25 50.8) (xy 96.52 50.8))
+  (wire (pts (xy 74.93 60.96) (xy 74.93 63.5))
+    (stroke (width 0) (type default))
+  )
+  (wire (pts (xy 95.25 50.8) (xy 99.06 50.8))
     (stroke (width 0) (type default))
   )
@@
     (stroke (width 0) (type default))
   )
-  (wire (pts (xy 74.93 73.66) (xy 87.63 73.66))
+  (wire (pts (xy 74.93 73.66) (xy 83.82 73.66))
+    (stroke (width 0) (type default))
+  )
+  (wire (pts (xy 106.68 60.96) (xy 111.76 60.96))
     (stroke (width 0) (type default))
   )
@@
   )
   (wire (pts (xy 118.11 127) (xy 120.65 127))
+    (stroke (width 0) (type default))
+  )
+  (wire (pts (xy 74.93 71.12) (xy 74.93 73.66))
     (stroke (width 0) (type default))
   )
@@
     (effects (font (size 1.27 1.27)) (justify right))
   )
-  (hierarchical_label "GPIO_BUTTON_CHECK" (shape input) (at 96.52 50.8 0) (fields_autoplaced)
+  (hierarchical_label "GPIO_BUTTON_CHECK" (shape input) (at 99.06 50.8 0) (fields_autoplaced)
     (effects (font (size 1.27 1.27)) (justify left))
   )
@@
     (effects (font (size 1.27 1.27)) (justify right))
   )
-  (hierarchical_label "GPIO_POWEROFF" (shape input) (at 96.52 54.61 0) (fields_autoplaced)
+  (hierarchical_label "GPIO_POWEROFF" (shape input) (at 99.06 54.61 0) (fields_autoplaced)
     (effects (font (size 1.27 1.27)) (justify left))
   )
@@
       (effects (font (size 1.27 1.27)) (justify left))
     )
-    (property "Value" "100n" (at 52.07 48.26 0)
+    (property "Value" "100nF" (at 52.07 48.26 0)
       (effects (font (size 1.27 1.27)) (justify left))
     )
@@
     )
   )
+  (symbol (lib_id "Switch:SW_DPST") (at 109.22 66.04 90) (unit 1)
+    (in_bom yes) (on_board yes) (dnp no) (fields_autoplaced)
+    (property "Reference" "SW4" (at 114.3 64.77 90)
+      (effects (font (size 1.27 1.27)) (justify right))
+    )
+    (property "Value" "SW_DPST" (at 114.3 67.31 90)
+      (effects (font (size 1.27 1.27)) (justify right))
+    )
+    (property "Footprint" "Button_Switch_SMD:SW_Push_1P1T_NO_6x6mm_H9.5mm" (at 109.22 66.04 0)
+      (effects (font (size 1.27 1.27)) hide)
+    )
+    (property "Datasheet" "~" (at 109.22 66.04 0)
+      (effects (font (size 1.27 1.27)) hide)
+    )
+    (pin "1")
+    (pin "3")
+    (pin "2")
+    (pin "4")
+    (instances
+      (project "grip_strength_meter"
+        (path "/1f4b217c-5456-4c03-a123-3ef9839449c6/4e936500-8830-4ef1-9c08-090defb3e135"
+          (reference "SW4") (unit 1)
+        )
+      )
+    )
+  )
   (symbol (lib_id "Device:R") (at 93.98 163.83 270) (unit 1)
     (in_bom yes) (on_board yes) (dnp no)
@@
     )
   )
-  (symbol (lib_id "Device:R") (at 91.44 73.66 270) (unit 1)
-    (in_bom yes) (on_board yes) (dnp no) (fields_autoplaced)
-    (property "Reference" "R40" (at 91.44 67.31 90)
-      (effects (font (size 1.27 1.27)))
-    )
-    (property "Value" "100R" (at 91.44 69.85 90)
-      (effects (font (size 1.27 1.27)))
-    )
-    (property "Footprint" "Resistor_SMD:R_0805_2012Metric" (at 91.44 71.882 90)
-      (effects (font (size 1.27 1.27)) hide)
-    )
-    (property "Datasheet" "~" (at 91.44 73.66 0)
+  (symbol (lib_id "Device:R") (at 87.63 73.66 270) (unit 1)
+    (in_bom yes) (on_board yes) (dnp no) (fields_autoplaced)
+    (property "Reference" "R40" (at 87.63 67.31 90)
+      (effects (font (size 1.27 1.27)))
+    )
+    (property "Value" "100R" (at 87.63 69.85 90)
+      (effects (font (size 1.27 1.27)))
+    )
+    (property "Footprint" "Resistor_SMD:R_0805_2012Metric" (at 87.63 71.882 90)
+      (effects (font (size 1.27 1.27)) hide)
+    )
+    (property "Datasheet" "~" (at 87.63 73.66 0)
       (effects (font (size 1.27 1.27)) hide)
     )
@@
     )
   )
-  (symbol (lib_id "Device:R") (at 74.93 69.85 0) (unit 1)
-    (in_bom yes) (on_board yes) (dnp no) (fields_autoplaced)
-    (property "Reference" "R39" (at 77.47 68.5799 0)
-      (effects (font (size 1.27 1.27)) (justify left))
-    )
-    (property "Value" "1M" (at 77.47 71.1199 0)
-      (effects (font (size 1.27 1.27)) (justify left))
-    )
-    (property "Footprint" "Resistor_SMD:R_0805_2012Metric" (at 73.152 69.85 90)
-      (effects (font (size 1.27 1.27)) hide)
-    )
-    (property "Datasheet" "~" (at 74.93 69.85 0)
+  (symbol (lib_id "Device:R") (at 74.93 67.31 0) (unit 1)
+    (in_bom yes) (on_board yes) (dnp no) (fields_autoplaced)
+    (property "Reference" "R39" (at 77.47 66.0399 0)
+      (effects (font (size 1.27 1.27)) (justify left))
+    )
+    (property "Value" "1M" (at 77.47 68.5799 0)
+      (effects (font (size 1.27 1.27)) (justify left))
+    )
+    (property "Footprint" "Resistor_SMD:R_0805_2012Metric" (at 73.152 67.31 90)
+      (effects (font (size 1.27 1.27)) hide)
+    )
+    (property "Datasheet" "~" (at 74.93 67.31 0)
       (effects (font (size 1.27 1.27)) hide)
     )
@@
         )
       )
-    )
-  )
-  (symbol (lib_id "TS-1187A-B-A-B:TS-1187A-B-A-B") (at 101.6 66.04 270) (unit 1)
-    (in_bom yes) (on_board yes) (dnp no) (fields_autoplaced)
-    (property "Reference" "S3" (at 105.41 64.77 90)
-      (effects (font (size 1.27 1.27)) (justify left))
-    )
-    (property "Value" "TS-1187A-B-A-B" (at 105.41 67.31 90)
-      (effects (font (size 1.27 1.27)) (justify left))
-    )
-    (property "Footprint" "TS-1187A-B-A-B:SW_TS-1187A-B-A-B" (at 101.6 66.04 0)
-      (effects (font (size 1.27 1.27)) (justify bottom) hide)
-    )
-    (property "Datasheet" "" (at 101.6 66.04 0)
-      (effects (font (size 1.27 1.27)) hide)
-    )
-    (property "PARTREV" "A0" (at 101.6 66.04 0)
-      (effects (font (size 1.27 1.27)) (justify bottom) hide)
-    )
-    (property "MANUFACTURER" "XKB Industrial Precision" (at 101.6 66.04 0)
-      (effects (font (size 1.27 1.27)) (justify bottom) hide)
-    )
-    (property "MAXIMUM_PACKAGE_HEIGHT" "1.5mm" (at 101.6 66.04 0)
-      (effects (font (size 1.27 1.27)) (justify bottom) hide)
-    )
-    (property "STANDARD" "Manufacturer Recommendations" (at 101.6 66.04 0)
-      (effects (font (size 1.27 1.27)) (justify bottom) hide)
-    )
-    (pin "A")
-    (pin "B")
-    (pin "C")
-    (pin "D")
-    (instances
-      (project "grip_strength_meter"
-        (path "/1f4b217c-5456-4c03-a123-3ef9839449c6/4e936500-8830-4ef1-9c08-090defb3e135"
-          (reference "S3") (unit 1)
-        )
-      )

Commit message: minor fix
Other:
- note added: "Must be like 100K and 100K because of esp32 adc parameters"
- note added: "We can add charge detection schematic, connect STDBY and CHRGE to 3v3 through R and then connect to gpio mcu pins. like here https://electronics.stackexchange.com/questions/657473/is-it-possible-to-interface-the-tp4056-charge-ic-with-a-mcu"
- note added: "We need to add 10 uF C between bat+ and bat-"
- note added: "Очень важная заметка! При проектировании цепи включения нужно помнить что по каким-то неясным причинам затвор Q7 не может сам быстро разрядиться через R39 и закрыть Q7. Из-за этого любой шум на пине GPIO_POWEROFF приводит к открытию Q7, что приводит к запитыванию всей схемы ЭТО ОЧЕНЬ ПЛОХО, потому что вводит всю схему в цикл бесконечных перезагрузок: Q7 закрывается->питание на МК пропадает->GPIO_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"
- note added: "Поэтому можно хардварно улучшать схему, но на данный момент: 1) поставить перемычку для самой первой прошивки схемы 2) поставить в параллель с R39 кондер на 1 мкФ или больше, он все делает хорошо"
- note added: "При перепрошивке приходится постоянно зажимать кнопку POWER, перемычка была бы удобнее"
- note added: "ТУТ НУЖЕН КОНДЕР НА 1-10мкФ В ПАРАЛЛЕЛЬ С R39 (2u2 норм)"
- note added: "собственно наверно лучше было бы если питание 5в всегда включало девайс а кнопка нужна была бы только при работе с аккумом надо это обдумать"
- note removed: "Do we need that resistor?"
- moved on the sheet: R36, R37
Changed lines of the file:
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@@
   (junction (at 124.46 41.91) (diameter 0) (color 0 0 0 0)
   )
-  (junction (at 93.98 109.22) (diameter 0) (color 0 0 0 0)
+  (junction (at 243.84 139.7) (diameter 0) (color 0 0 0 0)
   )
   (junction (at 132.08 127) (diameter 0) (color 0 0 0 0)
@@
     (stroke (width 0) (type default))
   )
-  (wire (pts (xy 93.98 107.95) (xy 93.98 109.22))
+  (wire (pts (xy 243.84 138.43) (xy 243.84 139.7))
     (stroke (width 0) (type default))
   )
@@
     (stroke (width 0) (type default))
   )
-  (wire (pts (xy 93.98 109.22) (xy 93.98 110.49))
+  (wire (pts (xy 243.84 139.7) (xy 243.84 140.97))
     (stroke (width 0) (type default))
   )
@@
     (stroke (width 0) (type default))
   )
-  (wire (pts (xy 91.44 109.22) (xy 93.98 109.22))
+  (wire (pts (xy 241.3 139.7) (xy 243.84 139.7))
     (stroke (width 0) (type default))
   )
@@
     (stroke (width 0) (type default))
   )
-  (wire (pts (xy 93.98 118.11) (xy 93.98 121.92))
-    (stroke (width 0) (type default))
-  )
-  (wire (pts (xy 93.98 96.52) (xy 93.98 100.33))
+  (wire (pts (xy 243.84 148.59) (xy 243.84 152.4))
+    (stroke (width 0) (type default))
+  )
+  (wire (pts (xy 243.84 127) (xy 243.84 130.81))
     (stroke (width 0) (type default))
   )
@@
     (stroke (width 0) (type default))
   )
+  (text "собственно наверно лучше было бы если питание 5в всегда включало девайс\nа кнопка нужна была бы только при работе с аккумом\nнадо это обдумать"
+    (at 121.92 88.9 0)
+    (effects (font (size 1.27 1.27)) (justify left bottom))
+  )
   (text "must be pulled up" (at 101.6 49.53 0)
     (effects (font (size 1.27 1.27)) (justify left bottom))
@@
   )
   (text "https://www.best-microcontroller-projects.com/dw01a.html"
-    (at 54.61 185.42 0)
-    (effects (font (size 1.27 1.27)) (justify left bottom))
-  )
-  (text "Do we need that resistor?" (at 129.54 50.8 0)
+    (at 54.61 184.15 0)
     (effects (font (size 1.27 1.27)) (justify left bottom))
   )
@@
     (effects (font (size 1.27 1.27)) (justify left bottom))
   )
+  (text "We can add charge detection schematic, \nconnect STDBY and CHRGE to 3v3 through R and then connect\nto gpio mcu pins.\nlike here\nhttps://electronics.stackexchange.com/questions/657473/is-it-possible-to-interface-the-tp4056-charge-ic-with-a-mcu"
+    (at 21.59 109.22 0)
+    (effects (font (size 1.27 1.27)) (justify left bottom))
+  )
+  (text "Поэтому можно хардварно улучшать схему, но на данный момент:\n1) поставить перемычку для самой первой прошивки схемы\n2) поставить в параллель с R39 кондер на 1 мкФ или больше,\nон все делает хорошо\n"
+    (at 134.62 66.04 0)
+    (effects (font (size 1.27 1.27)) (justify left bottom))
+  )
+  (text "We need to add 10 uF C between bat+ and bat-" (at 118.11 173.99 0)
+    (effects (font (size 1.27 1.27)) (justify left bottom))
+  )
   (text "Voltage divider to measure\nv batt on esp adc, to show to user"
-    (at 74.93 92.71 0)
+    (at 220.98 121.92 0)
     (effects (font (size 1.27 1.27)) (justify left bottom))
   )
@@
     (effects (font (size 1.27 1.27)) (justify left bottom))
   )
+  (text "Must be like 100K and 100K \nbecause of esp32 adc parameters"
+    (at 245.11 130.81 0)
+    (effects (font (size 1.27 1.27)) (justify left bottom))
+  )
   (text "LI-Po charger" (at 63.5 130.81 0)
     (effects (font (size 1.27 1.27)) (justify left bottom))
@@
     (effects (font (size 1.27 1.27)) (justify left bottom))
   )
+  (text "Очень важная заметка!\nПри проектировании цепи включения нужно помнить \nчто по каким-то неясным причинам затвор Q7 не может сам быстро разрядиться\nчерез R39 и закрыть Q7. Из-за этого любой шум на пине GPIO_POWEROFF\nприводит к открытию Q7, что приводит к запитыванию всей схемы\nЭТО ОЧЕНЬ ПЛОХО, потому что вводит всю схему в цикл бесконечных перезагрузок:\nQ7 закрывается->питание на МК пропадает->GPIO_POWEROFF начинает шуметь->\nшум открывает Q7->мк включается->Q7 закрывается и все по-новой "
+    (at 91.44 35.56 0)
+    (effects (font (size 1.27 1.27) (thickness 0.254) bold) (justify left bottom))
+  )
   (text "Power selector \nscheme" (at 114.3 119.38 0)
     (effects (font (size 1.27 1.27)) (justify left bottom))
   )
+  (text "ТУТ НУЖЕН КОНДЕР НА 1-10мкФ В ПАРАЛЛЕЛЬ С R39 (2u2 норм)"
+    (at 62.23 77.47 0)
+    (effects (font (size 1.27 1.27) bold) (justify left bottom))
+  )
   (text "G" (at 132.08 133.35 0)
     (effects (font (size 1.27 1.27)) (justify left bottom))
+  )
+  (text "При перепрошивке приходится постоянно зажимать кнопку POWER, перемычка была бы удобнее\n"
+    (at 62.23 81.28 0)
+    (effects (font (size 1.27 1.27) bold) (justify left bottom))
   )
   (text "Main power supply\nfrom Li-Po/USB to 3v3 " (at 157.48 128.27 0)
@@
     )
   )
-  (hierarchical_label "V_BAT" (shape input) (at 93.98 96.52 180) (fields_autoplaced)
+  (hierarchical_label "V_BAT" (shape input) (at 243.84 127 180) (fields_autoplaced)
     (effects (font (size 1.27 1.27)) (justify right))
   )
@@
     (effects (font (size 1.27 1.27)) (justify right))
   )
-  (hierarchical_label "GND" (shape input) (at 93.98 121.92 180) (fields_autoplaced)
+  (hierarchical_label "GND" (shape input) (at 243.84 152.4 180) (fields_autoplaced)
     (effects (font (size 1.27 1.27)) (justify right))
   )
@@
     (effects (font (size 1.27 1.27)) (justify right))
   )
-  (hierarchical_label "V_BAT_MEASURE" (shape input) (at 91.44 109.22 180) (fields_autoplaced)
+  (hierarchical_label "V_BAT_MEASURE" (shape input) (at 241.3 139.7 180) (fields_autoplaced)
     (effects (font (size 1.27 1.27)) (justify right))
   )
@@
     )
   )
-  (symbol (lib_id "Device:R") (at 93.98 114.3 0) (unit 1)
+  (symbol (lib_id "Device:R") (at 243.84 144.78 0) (unit 1)
     (in_bom yes) (on_board yes) (dnp no) (fields_autoplaced)
-    (property "Reference" "R37" (at 96.52 113.03 0)
+    (property "Reference" "R37" (at 246.38 143.51 0)
       (effects (font (size 1.27 1.27)) (justify left))
     )
-    (property "Value" "30K" (at 96.52 115.57 0)
+    (property "Value" "30K" (at 246.38 146.05 0)
       (effects (font (size 1.27 1.27)) (justify left))
     )
-    (property "Footprint" "Resistor_SMD:R_0805_2012Metric" (at 92.202 114.3 90)
+    (property "Footprint" "Resistor_SMD:R_0805_2012Metric" (at 242.062 144.78 90)
       (effects (font (size 1.27 1.27)) hide)
     )
-    (property "Datasheet" "~" (at 93.98 114.3 0)
+    (property "Datasheet" "~" (at 243.84 144.78 0)
       (effects (font (size 1.27 1.27)) hide)
     )
@@
     )
   )
-  (symbol (lib_id "Device:R") (at 93.98 104.14 0) (unit 1)
+  (symbol (lib_id "Device:R") (at 243.84 134.62 0) (unit 1)
     (in_bom yes) (on_board yes) (dnp no) (fields_autoplaced)
-    (property "Reference" "R36" (at 96.52 102.87 0)
+    (property "Reference" "R36" (at 246.38 133.35 0)
       (effects (font (size 1.27 1.27)) (justify left))
     )
-    (property "Value" "10K" (at 96.52 105.41 0)
+    (property "Value" "10K" (at 246.38 135.89 0)
       (effects (font (size 1.27 1.27)) (justify left))
     )
-    (property "Footprint" "Resistor_SMD:R_0805_2012Metric" (at 92.202 104.14 90)
+    (property "Footprint" "Resistor_SMD:R_0805_2012Metric" (at 242.062 134.62 90)
       (effects (font (size 1.27 1.27)) hide)
     )
-    (property "Datasheet" "~" (at 93.98 104.14 0)
+    (property "Datasheet" "~" (at 243.84 134.62 0)
       (effects (font (size 1.27 1.27)) hide)
     )
